File: RockLight.kicad_sch (KiCad schematic)
At the start: 17 parts, among them J1 USB_C_Receptacle_USB2.0_16P, J2 ISP, SW1 USER, SW2 RESET, U1 ATtiny85-10SU

Commit message: Add project files
Parts:
- added JP1: Jumper_2_Small_Open, Jumper:SolderJumper-2_P1.3mm_Open_TrianglePad1.0x1.5mm, symbol Jumper:Jumper_2_Small_Open
- added R3: 10k, Resistor_SMD:R_0402_1005Metric, symbol Device:R_Small_US
- added TP1: SIG, TestPoint:TestPoint_Pad_D1.5mm, symbol Connector:TestPoint
- added TP2: +5V, TestPoint:TestPoint_Pad_D1.5mm, symbol Connector:TestPoint
- added TP3: GND, TestPoint:TestPoint_Pad_D1.5mm, symbol Connector:TestPoint
- J2: footprint Connector_PinHeader_2.54mm:PinHeader_1x06_P2.54mm_Vertical -> Connector_JST:JST_PH_B6B-PH-K_1x06_P2.00mm_Vertical
Connections:
- net +5V: now also JP1.2 (B), R3.1, TP2.1; no longer D1.1 (VDD), D2.1 (VDD), D3.1 (VDD), D4.1 (VDD)
- net GND: now also TP3.1
- net RESET: now also R3.2
- net at D1.4 (DIN), U1.2 (XTAL1/PB3): now also TP1.1
- new net: D1.1 (VDD), D2.1 (VDD), D3.1 (VDD), D4.1 (VDD), JP1.1 (A)
Other:
- moved on the sheet: H1, H2, H3, H4
